Commit message: changed caster wheels into spheres

File: my_rb1_description/urdf/my_rb1_robot.urdf (robot description, URDF)
Before this commit: robot rb1_robot, 7 links, 6 joints
Links:
- link back_caster: geometry collision sphere radius=0.025; visual sphere radius=0.025
- link front_caster: geometry collision sphere radius=0.025; visual sphere radius=0.025
